Commit message: Fix path to meshes in urdf and refactoring tuto inverse kinematics

File: models/romeo_small.urdf (robot description, URDF)
Before this commit: robot romeoH37V1, 34 links, 33 joints
Links:
- link HeadRollLink: geometry collision mesh filename=package://meshes/collision/HeadRoll.dae scale=1 1 1; visual mesh filename=package://meshes/visual/HeadRoll.dae scale=1 1 1
- link LElbowYawLink: geometry collision mesh filename=package://meshes/collision/LElbowYaw.dae scale=1 1 1; visual mesh filename=package://meshes/visual/LElbowYaw.dae scale=1 1 1
- link LHipPitchLink: geometry collision mesh filename=package://meshes/collision/LHipPitch.dae scale=1 1 1; visual mesh filename=package://meshes/visual/LHipPitch.dae scale=1 1 1
- link LKneePitchLink: geometry collision mesh filename=package://meshes/collision/LKneePitch.dae scale=1 1 1; visual mesh filename=package://meshes/visual/LKneePitch.dae scale=1 1 1
- link LShoulderYawLink: geometry collision mesh filename=package://meshes/collision/LShoulderYaw.dae scale=1 1 1; visual mesh filename=package://meshes/visual/LShoulderYaw.dae scale=1 1 1
- link LWristRollLink: geometry collision mesh filename=package://meshes/collision/LWristRoll.dae scale=1 1 1; visual mesh filename=package://meshes/visual/LWristRoll.dae scale=1 1 1
- link LWristYawLink: geometry collision mesh filename=package://meshes/collision/LWristYaw.dae scale=1 1 1; visual mesh filename=package://meshes/visual/LWristYaw.dae scale=1 1 1
- link NeckPitchLink: geometry collision mesh filename=package://meshes/collision/NeckPitch.dae scale=1 1 1; visual mesh filename=package://meshes/visual/NeckPitch.dae scale=1 1 1
- link RElbowYawLink: geometry collision mesh filename=package://meshes/collision/RElbowYaw.dae scale=1 1 1; visual mesh filename=package://meshes/visual/RElbowYaw.dae scale=1 1 1
- link RHipPitchLink: geometry collision mesh filename=package://meshes/collision/RHipPitch.dae scale=1 1 1; visual mesh filename=package://meshes/visual/RHipPitch.dae scale=1 1 1
- link RKneePitchLink: geometry collision mesh filename=package://meshes/collision/RKneePitch.dae scale=1 1 1; visual mesh filename=package://meshes/visual/RKneePitch.dae scale=1 1 1
- link RShoulderYawLink: geometry collision mesh filename=package://meshes/collision/RShoulderYaw.dae scale=1 1 1; visual mesh filename=package://meshes/visual/RShoulderYaw.dae scale=1 1 1
- link RWristRollLink: geometry collision mesh filename=package://meshes/collision/RWristRoll.dae scale=1 1 1; visual mesh filename=package://meshes/visual/RWristRoll.dae scale=1 1 1
- link RWristYawLink: geometry collision mesh filename=package://meshes/collision/RWristYaw.dae scale=1 1 1; visual mesh filename=package://meshes/visual/RWristYaw.dae scale=1 1 1
- link body: geometry collision mesh filename=package://meshes/collision/TrunkYaw.dae scale=1 1 1; visual mesh filename=package://meshes/visual/TrunkYaw.dae scale=1 1 1
- link l_ankle: geometry collision mesh filename=package://meshes/collision/LAnkleRoll.dae scale=1 1 1; visual mesh filename=package://meshes/visual/LAnkleRoll.dae scale=1 1 1
- link l_wrist: geometry collision mesh filename=package://meshes/collision/LWristPitch.dae scale=1 1 1; visual mesh filename=package://meshes/visual/LWristPitch.dae scale=1 1 1
- link r_ankle: geometry collision mesh filename=package://meshes/collision/RAnkleRoll.dae scale=1 1 1; visual mesh filename=package://meshes/visual/RAnkleRoll.dae scale=1 1 1
- link r_wrist: geometry collision mesh filename=package://meshes/collision/RWristPitch.dae scale=1 1 1; visual mesh filename=package://meshes/visual/RWristPitch.dae scale=1 1 1
- link torso: geometry collision mesh filename=package://meshes/collision/Torso.dae scale=1 1 1; visual mesh filename=package://meshes/visual/Torso.dae scale=1 1 1
