Commit message: Adapted both the urdf parser and the romeo model to enable romeo inside pinocchio. CAUTION: Romeo is not standard any more and should be corrected, by enabling fixed joint in the urdf parser.

File: models/romeo.urdf (robot description, URDF)
Before this commit: robot romeo, 70 links, 69 joints
Joints:
- joint LEyePitch: type revolute -> fixed
- joint LEyeYaw: type revolute -> fixed
- joint LFinger11: type revolute -> fixed
- joint LFinger12: type revolute -> fixed
- joint LFinger13: type revolute -> fixed
- joint LFinger21: type revolute -> fixed
- joint LFinger22: type revolute -> fixed
- joint LFinger23: type revolute -> fixed
- joint LFinger31: type revolute -> fixed
- joint LFinger32: type revolute -> fixed
- joint LFinger33: type revolute -> fixed
- joint LHipYaw: parent body -> base_link
- joint LThumb1: type revolute -> fixed
- joint LThumb2: type revolute -> fixed
- joint LThumb3: type revolute -> fixed
- joint REyePitch: type revolute -> fixed
- joint REyeYaw: type revolute -> fixed
- joint RFinger11: type revolute -> fixed
- joint RFinger12: type revolute -> fixed
- joint RFinger13: type revolute -> fixed
- joint RFinger21: type revolute -> fixed
- joint RFinger22: type revolute -> fixed
- joint RFinger23: type revolute -> fixed
- joint RFinger31: type revolute -> fixed
- joint RFinger32: type revolute -> fixed
- joint RFinger33: type revolute -> fixed
- joint RHipYaw: parent body -> base_link
- joint RThumb1: type revolute -> fixed
- joint RThumb2: type revolute -> fixed
- joint RThumb3: type revolute -> fixed
- joint TrunkYaw: parent body -> base_link

Commit message: [bench][unittest] Reworked the comparison test between pinocchio and hpp : more tests for benchmarks along with functional tests ; removing magic paths to urdf models + modification of romeo urdf model. Also added a specific BUILD_TESTS_WITH_HPP cmake variable. If you want to run tests that execute hpp robot loading, be sure to have the package romeo_pinocchio installed (it is just a package done done by hand for the moment)

File: models/romeo.urdf (robot description, URDF)
Before this commit: robot romeoH37V1, 34 links, 33 joints
Links:
- added link base_link
Joints:
- added joint waist: type fixed, parent base_link, child body, origin xyz=0 0 0 rpy=0 0 0
