Commit message: Atlas robot with shadow hands

File: models/atlas_with_srs.urdf (robot description, URDF)
Before this commit: robot drc_skeleton, 79 links, 78 joints
Links:
- link sr_left_index_finger_distal: mass None -> 0.648
- link sr_left_index_finger_knuckle: mass None -> 0.648
- link sr_left_index_finger_middle: mass None -> 0.648
- link sr_left_index_finger_proximal: mass None -> 0.648
- link sr_left_little_finger_distal: mass None -> 0.648
- link sr_left_little_finger_knuckle: mass None -> 0.648
- link sr_left_little_finger_metacarpal: mass None -> 0.648
- link sr_left_little_finger_middle: mass None -> 0.648
- link sr_left_little_finger_proximal: mass None -> 0.648
- link sr_left_middle_finger_distal: mass None -> 0.648
- link sr_left_middle_finger_knuckle: mass None -> 0.648
- link sr_left_middle_finger_middle: mass None -> 0.648
- link sr_left_middle_finger_proximal: mass None -> 0.648
- link sr_left_palm: mass None -> 0.648
- link sr_left_ring_finger_distal: mass None -> 0.648
- link sr_left_ring_finger_knuckle: mass None -> 0.648
- link sr_left_ring_finger_middle: mass None -> 0.648
- link sr_left_ring_finger_proximal: mass None -> 0.648
- link sr_left_thumb_distal: mass None -> 0.648
- link sr_left_thumb_middle: mass None -> 0.648
- link sr_left_thumb_proximal: mass None -> 0.648
- link sr_left_wrist: mass None -> 0.648
- link sr_right_index_finger_distal: mass None -> 0.648
- link sr_right_index_finger_knuckle: mass None -> 0.648
- link sr_right_index_finger_middle: mass None -> 0.648
- link sr_right_index_finger_proximal: mass None -> 0.648
- link sr_right_little_finger_distal: mass None -> 0.648
- link sr_right_little_finger_knuckle: mass None -> 0.648
- link sr_right_little_finger_metacarpal: mass None -> 0.648
- link sr_right_little_finger_middle: mass None -> 0.648
- link sr_right_little_finger_proximal: mass None -> 0.648
- link sr_right_middle_finger_distal: mass None -> 0.648
- link sr_right_middle_finger_knuckle: mass None -> 0.648
- link sr_right_middle_finger_middle: mass None -> 0.648
- link sr_right_middle_finger_proximal: mass None -> 0.648
- link sr_right_palm: mass None -> 0.648
- link sr_right_ring_finger_distal: mass None -> 0.648
- link sr_right_ring_finger_knuckle: mass None -> 0.648
- link sr_right_ring_finger_middle: mass None -> 0.648
- link sr_right_ring_finger_proximal: mass None -> 0.648
- link sr_right_thumb_distal: mass None -> 0.648
- link sr_right_thumb_middle: mass None -> 0.648
- link sr_right_thumb_proximal: mass None -> 0.648
- link sr_right_wrist: mass None -> 0.648
